Commit message: Added

File: models/simple_arm.urdf (robot description, URDF)
Before this commit: robot simple_arm, 5 links, 4 joints
Links:
- added link link4, mass 0.1; collision box size=0.025 0.025 0.05; visual box size=0.025 0.025 0.05
- added link slider_link, mass 2.0; collision cylinder length=0.04 radius=0.06; visual cylinder length=0.04 radius=0.06
- link base_link: mass 1.0 -> 5.0; geometry collision box size=1.2 0.1 0.02; visual box size=1.2 0.1 0.02
- link link3: geometry collision box size=0.03 0.03 0.10; visual box size=0.03 0.03 0.10
Joints:
- removed joint wrist_to_ee
- added joint base_rail: type prismatic, parent base_link, child slider_link, origin xyz=0 0 0.02 rpy=0 0 0, axis 1 0 0, limit lower=-0.5 upper=0.5 effort=100.0 velocity=1.0
- added joint wrist_pitch: type revolute, parent link3, child link4, origin xyz=0 0 0.10 rpy=0 0 0, axis 0 1 0, limit lower=-1.5708 upper=1.5708 effort=5.0 velocity=1.5
- added joint wrist_roll: type revolute, parent link4, child end_effector, origin xyz=0 0 0.05 rpy=0 0 0, axis 0 0 1, limit lower=-3.14159 upper=3.14159 effort=3.0 velocity=2.0
- joint shoulder_pan: origin xyz=0 0 0.05 rpy=0 0 0 -> xyz=0 0 0.04 rpy=0 0 0; parent base_link -> slider_link
